Commit message: Created core URDF

File: vektor_pkg/description/vektor.xacro (robot description, xacro)
@@ -1,4 +1,4 @@
 <?xml version="1.1" encoding="UTF-8"?>
 <robot name="vektor" xmlns:xacro="http://www.ros.org/wiki/xacro">
-    <link name="base_link"></link>
+    <xacro:include filename="vektor_core.xacro"/>
 </robot>

Commit message: Created simulation

File: vektor_pkg/description/vektor.xacro (robot description, xacro)
@@ -2,3 +2,4 @@
 <robot name="vektor" xmlns:xacro="http://www.ros.org/wiki/xacro">
     <xacro:include filename="vektor_core.xacro"/>
+    <xacro:include filename="gazebo_control.xacro"/>
 </robot>

File: vektor_pkg/description/vektor_core.xacro (robot description, xacro)
@@ -41,4 +41,7 @@
         </xacro:inertial_box>
     </link>
+    <gazebo reference="chassis_link">
+        <material>Gazebo/White</material>
+    </gazebo>
     <!-- LEFT WHEEL LINK -->
     <joint name="left_wheel_joint" type="continuous">
@@ -64,4 +67,7 @@
         </xacro:inertial_cylinder>
     </link>
+    <gazebo reference="left_wheel_link">
+        <material>Gazebo/Blue</material>
+    </gazebo>
     <!-- RIGHT WHEEL LINK -->
     <joint name="right_wheel_joint" type="continuous">
@@ -87,4 +93,7 @@
         </xacro:inertial_cylinder>
     </link>
+    <gazebo reference="right_wheel_link">
+        <material>Gazebo/Blue</material>
+    </gazebo>
     <!-- CASTER WHEEL LINK -->
     <joint name="caster_wheel_joint" type="fixed">
@@ -109,3 +118,8 @@
         </xacro:inertial_sphere>
     </link>
+    <gazebo reference="caster_wheel_link">
+        <material>Gazebo/Black</material>
+        <mu1 value="0.001"/>
+        <mu2 value="0.001"/>
+    </gazebo>
 </robot>
