Commit message: fixed ignition launcher and added lidar sensor

File: vektor_pkg/description/gazebo_control.xacro (robot description, xacro)
@@ -2,19 +2,18 @@
 <robot xmlns:xacro="http://www.ros.org/wiki/xacro">
     <gazebo>
-        <plugin name="diff_drive" filename="libgazebo_ros_diff_drive.so">
-            <!-- WHEEL INFORMATION -->
+        <plugin
+            filename="libignition-gazebo-diff-drive-system.so"
+            name="ignition::gazebo::systems::DiffDrive">
             <left_joint>left_wheel_joint</left_joint>
             <right_joint>right_wheel_joint</right_joint>
             <wheel_separation>0.35</wheel_separation>
-            <wheel_diameter>0.1</wheel_diameter>
-            <!-- LIMITS -->
-            <max_wheel_torque>200</max_wheel_torque>
-            <max_wheel_acceleration>10.0</max_wheel_acceleration>
-            <!-- OUTPUT-->
-            <odometry_frame>odom</odometry_frame>
-            <robot_base_frame>base_link</robot_base_frame>
-            <publish_odom>true</publish_odom>
-            <publish_odom_tf>true</publish_odom_tf>
-            <publish_wheel_tf>true</publish_wheel_tf>
+            <wheel_radius>0.05</wheel_radius>
+            <odom_publish_frequency>1</odom_publish_frequency>
+            <topic>cmd_vel</topic>
+        </plugin>
+        <plugin
+            filename="libignition-gazebo-sensors-system.so"
+            name="ignition::gazebo::systems::Sensors">
+            <render_engine>ogre2</render_engine>
         </plugin>
     </gazebo>

File: vektor_pkg/description/lidar.xacro (robot description, xacro)
@@ -7,9 +7,12 @@
     </joint>
     <link name="lidar_frame">
+        <frame_id>lidar_frame</frame_id>
         <visual>
             <geometry>
                 <cylinder radius="0.05" length="0.04"/>
             </geometry>
-            <material name="Olive"/>
+            <material name="red2">
+                <color rgba="1.0 0.0 0.0 1.0"/>
+            </material>
         </visual>
         <collision>
@@ -23,8 +26,8 @@
     </link>
     <gazebo reference="lidar_frame">
-        <material>Gazebo/Green</material>
-        <sensor name="lidar" type="ray">
-            <pose> 0 0 0 0 0 0 </pose>
-            <visualize>true</visualize>
+        <sensor name='lidar_frame' type='gpu_lidar'>
+            <pose>0 0 0 0 0 0</pose>
+            <topic>lidar</topic>
+            <ignition_frame_id>lidar_frame</ignition_frame_id>
             <update_rate>10</update_rate>
             <ray>
@@ -39,15 +42,10 @@
                 <range>
                     <min>0.3</min>
-                    <max>12</max>
+                    <max>5.0</max>
                     <resolution>0.01</resolution>
                 </range>
             </ray>
-            <plugin name="lidar_controller" filename="libgazebo_ros_ray_sensor.so">
-                <ros>
-                    <argument>~/out:=scan</argument>
-                </ros>
-                <output_type>sensor_msgs/LaserScan</output_type>
-                <frame_name>lidar_frame</frame_name>
-            </plugin>
+            <always_on>1</always_on>
+            <visualize>true</visualize>
         </sensor>
     </gazebo>

File: vektor_pkg/description/materials.xacro (robot description, xacro)
@@ -49,3 +49,21 @@
         <color rgba="0.6 0.6 0.6 1"/>
     </material>
+    <material name="white">
+        <color rgba="1 1 1 1"/>
+    </material>
+    <material name="orange">
+        <color rgba="1 0.3 0.1 1"/>
+    </material>
+    <material name="blue">
+        <color rgba="0.2 0.2 1 1"/>
+    </material>
+    <material name="green">
+        <color rgba="0.2 1 0.2 1"/>
+    </material>
+    <material name="yellow">
+        <color rgba="1 1 0.2 1"/>
+    </material>
+    <material name="black">
+        <color rgba="0 0 0 1"/>
+    </material>
 </robot>

File: vektor_pkg/description/vektor.xacro (robot description, xacro)
@@ -5,4 +5,4 @@
     <xacro:include filename="lidar.xacro"/>
     <!-- <xacro:include filename="camera.xacro"/> -->
-    <xacro:include filename="depth_camera.xacro"/>
+    <!-- <xacro:include filename="depth_camera.xacro"/> -->
 </robot>

File: vektor_pkg/description/vektor_core.xacro (robot description, xacro)
@@ -1,27 +1,9 @@
 <?xml version="1.1" encoding="UTF-8"?>
 <robot xmlns:xacro="http://www.ros.org/wiki/xacro">
+    <!-- OTHER FILES -->
     <xacro:include filename="inertial_macros.xacro"/>
     <xacro:include filename="materials.xacro"/>
-    <material name="white">
-        <color rgba="1 1 1 1"/>
-    </material>
-    <material name="orange">
-        <color rgba="1 0.3 0.1 1"/>
-    </material>
-    <material name="blue">
-        <color rgba="0.2 0.2 1 1"/>
-    </material>
-    <material name="green">
-        <color rgba="0.2 1 0.2 1"/>
-    </material>
-    <material name="yellow">
-        <color rgba="1 1 0.2 1"/>
-    </material>
-    <material name="black">
-        <color rgba="0 0 0 1"/>
-    </material>
     <!-- BASE LINK -->
-    <link name="base_link">
-    </link>
+    <link name="base_link"/>
     <!-- CHASSIS LINK -->
     <joint name="chassis_joint" type="fixed">
@@ -48,7 +30,4 @@
         </xacro:inertial_box>
     </link>
-    <gazebo reference="chassis_link">
-        <material>Gazebo/White</material>
-    </gazebo>
     <!-- LEFT WHEEL LINK -->
     <joint name="left_wheel_joint" type="continuous">
@@ -63,5 +42,7 @@
                 <cylinder radius="0.05" length="0.04"/>
             </geometry>
-            <material name="Gold"/>
+            <material name="green2">
+                <color rgba="0.0 1.0 0.0 1.0"/>
+            </material>
         </visual>
         <collision>
@@ -74,7 +55,4 @@
         </xacro:inertial_cylinder>
     </link>
-    <gazebo reference="left_wheel_link">
-        <material>Gazebo/Blue</material>
-    </gazebo>
     <!-- RIGHT WHEEL LINK -->
     <joint name="right_wheel_joint" type="continuous">
@@ -89,5 +67,7 @@
                 <cylinder radius="0.05" length="0.04"/>
             </geometry>
-            <material name="Gold"/>
+            <material name="green2">
+                <color rgba="0.0 1.0 0.0 1.0"/>
+            </material>
         </visual>
         <collision>
@@ -100,7 +80,4 @@
         </xacro:inertial_cylinder>
     </link>
-    <gazebo reference="right_wheel_link">
-        <material>Gazebo/Blue</material>
-    </gazebo>
     <!-- CASTER WHEEL LINK -->
     <joint name="caster_wheel_joint" type="fixed">
@@ -114,5 +91,7 @@
                 <sphere radius="0.05"/>
             </geometry>
-            <material name="green"/>
+            <material name="blue2">
+                <color rgba="0.0 0.0 1.0 1.0"/>
+            </material>
         </visual>
         <collision>
@@ -126,5 +105,4 @@
     </link>
     <gazebo reference="caster_wheel_link">
-        <material>Gazebo/Black</material>
         <mu1 value="0.001"/>
         <mu2 value="0.001"/>
