Commit message: Initial LiDAR implementation

File: vektor_pkg/description/materials.xacro (robot description, xacro)
@@ -1,6 +1,51 @@
 <?xml version="1.1" encoding="UTF-8"?>
 <robot xmlns:xacro="http://www.ros.org/wiki/xacro">
-    <material name="white">
-        <color rgba="1 1 1 1"/>
+    <material name="pale-pink">
+        <color rgba="1 0.8 0.8 1"/>
+    </material>
+    <material name="pale-yellow">
+            <color rgba="1 1 0.6 1"/>
+    </material>
+    <material name="pale-blue">
+            <color rgba="0.7 0.7 1 1"/>
+    </material>
+    <material name="pale-green">
+            <color rgba="0.8 1 0.8 1"/>
+    </material>
+    <material name="Lavender">
+        <color rgba="0.7 0.5 0.9 1"/>
+    </material>
+    <material name="Light pink">
+        <color rgba="0.9 0.7 0.8 1"/>
+    </material>
+    <material name="Teal">
+        <color rgba="0.6 0.9 0.8 1"/>
+    </material>
+    <material name="Gold">
+        <color rgba="0.9 0.8 0.3 1"/>
+    </material>
+    <material name="Orange-red">
+        <color rgba="0.9 0.5 0.3 1"/>
+    </material>
+    <material name="Sky blue">
+        <color rgba="0.5 0.8 0.9 1"/>
+    </material>
+    <material name="Mint green">
+        <color rgba="0.7 0.9 0.7 1"/>
+    </material>
+    <material name="Salmon">
+        <color rgba="0.9 0.5 0.5 1"/>
+    </material>
+    <material name="Dark purple">
+        <color rgba="0.3 0.1 0.4 1"/>
+    </material>
+    <material name="Light blue">
+        <color rgba="0.5 0.7 0.9 1"/>
+    </material>
+    <material name="Olive">
+        <color rgba="0.5 0.6 0.3 1"/>
+    </material>
+    <material name="Gray">
+        <color rgba="0.6 0.6 0.6 1"/>
     </material>
 </robot>

File: vektor_pkg/description/vektor.xacro (robot description, xacro)
@@ -3,3 +3,4 @@
     <xacro:include filename="vektor_core.xacro"/>
     <xacro:include filename="gazebo_control.xacro"/>
+    <xacro:include filename="lidar.xacro"/>
 </robot>

File: vektor_pkg/description/vektor_core.xacro (robot description, xacro)
@@ -2,4 +2,5 @@
 <robot xmlns:xacro="http://www.ros.org/wiki/xacro">
     <xacro:include filename="inertial_macros.xacro"/>
+    <xacro:include filename="materials.xacro"/>
     <material name="white">
         <color rgba="1 1 1 1"/>
@@ -10,4 +11,10 @@
     <material name="blue">
         <color rgba="0.2 0.2 1 1"/>
+    </material>
+    <material name="green">
+        <color rgba="0.2 1 0.2 1"/>
+    </material>
+    <material name="yellow">
+        <color rgba="1 1 0.2 1"/>
     </material>
     <material name="black">
@@ -56,5 +63,5 @@
                 <cylinder radius="0.05" length="0.04"/>
             </geometry>
-            <material name="blue"/>
+            <material name="Gold"/>
         </visual>
         <collision>
@@ -82,5 +89,5 @@
                 <cylinder radius="0.05" length="0.04"/>
             </geometry>
-            <material name="blue"/>
+            <material name="Gold"/>
         </visual>
         <collision>
@@ -107,5 +114,5 @@
                 <sphere radius="0.05"/>
             </geometry>
-            <material name="black"/>
+            <material name="green"/>
         </visual>
         <collision>

Commit message: Fixed : on XML comment and minor adjusts

File: vektor_pkg/description/materials.xacro (robot description, xacro)
@@ -1,69 +1,38 @@
 <?xml version="1.1" encoding="UTF-8"?>
 <robot xmlns:xacro="http://www.ros.org/wiki/xacro">
-    <material name="pale-pink">
-        <color rgba="1 0.8 0.8 1"/>
-    </material>
-    <material name="pale-yellow">
-            <color rgba="1 1 0.6 1"/>
-    </material>
-    <material name="pale-blue">
-            <color rgba="0.7 0.7 1 1"/>
-    </material>
-    <material name="pale-green">
-            <color rgba="0.8 1 0.8 1"/>
-    </material>
-    <material name="Lavender">
-        <color rgba="0.7 0.5 0.9 1"/>
-    </material>
-    <material name="Light pink">
-        <color rgba="0.9 0.7 0.8 1"/>
-    </material>
-    <material name="Teal">
-        <color rgba="0.6 0.9 0.8 1"/>
-    </material>
-    <material name="Gold">
-        <color rgba="0.9 0.8 0.3 1"/>
-    </material>
-    <material name="Orange-red">
-        <color rgba="0.9 0.5 0.3 1"/>
-    </material>
-    <material name="Sky blue">
-        <color rgba="0.5 0.8 0.9 1"/>
-    </material>
-    <material name="Mint green">
-        <color rgba="0.7 0.9 0.7 1"/>
-    </material>
-    <material name="Salmon">
-        <color rgba="0.9 0.5 0.5 1"/>
-    </material>
-    <material name="Dark purple">
-        <color rgba="0.3 0.1 0.4 1"/>
-    </material>
-    <material name="Light blue">
-        <color rgba="0.5 0.7 0.9 1"/>
-    </material>
-    <material name="Olive">
-        <color rgba="0.5 0.6 0.3 1"/>
-    </material>
-    <material name="Gray">
-        <color rgba="0.6 0.6 0.6 1"/>
-    </material>
-    <material name="white">
-        <color rgba="1 1 1 1"/>
-    </material>
-    <material name="orange">
-        <color rgba="1 0.3 0.1 1"/>
-    </material>
-    <material name="blue">
-        <color rgba="0.2 0.2 1 1"/>
-    </material>
-    <material name="green">
-        <color rgba="0.2 1 0.2 1"/>
-    </material>
-    <material name="yellow">
-        <color rgba="1 1 0.2 1"/>
-    </material>
-    <material name="black">
-        <color rgba="0 0 0 1"/>
-    </material>
+  <!-- Solid -->
+  <material name="white">
+    <color rgba="1.0 1.0 1.0 1.0"/>
+  </material>
+  <material name="Gray">
+    <color rgba="0.6 0.6 0.6 1.0"/>
+  </material>
+  <material name="black">
+    <color rgba="0.0 0.0 0.0 1.0"/>
+  </material>
+  <material name="red">
+    <color rgba="1.0 0.0 0.0 1.0"/>
+  </material>
+  <material name="yellow">
+    <color rgba="1.0 1.0 0.0 1.0"/>
+  </material>
+  <material name="green">
+    <color rgba="0.0 1.0 0.0 1.0"/>
+  </material>
+  <material name="blue">
+    <color rgba="0.0 0.0 1.0 1.0"/>
+  </material>
+  <!-- Exotic -->
+  <material name="paper">
+    <color rgba="0.85 0.80 0.73 1.0"/>
+  </material>
+  <material name="Salmon">
+    <color rgba="0.9 0.5 0.5 1.0"/>
+  </material>
+  <material name="Dark purple">
+    <color rgba="0.3 0.1 0.4 1.0"/>
+  </material>
+  <material name="Olive">
+    <color rgba="0.5 0.6 0.3 1.0"/>
+  </material>
 </robot>

File: vektor_pkg/description/plugins.xacro (robot description, xacro)
@@ -47,5 +47,5 @@
       <topic>joint_states</topic>
       <!-- Custom topic on which this system will publish joint state messages. -->
-      <!-- TODO: SET PUBLISH FREQUENCY / UPDATE RATE. UNKNOWN TAG -->
+      <!-- [TODO] SET PUBLISH FREQUENCY / UPDATE RATE. UNKNOWN TAG. -->
       <!-- <joint_name>left_wheel_joint</joint_name> -->
       <!-- <joint_name>right_wheel_joint</joint_name> -->

File: vektor_pkg/description/vektor.xacro (robot description, xacro)
@@ -1,8 +1,8 @@
 <?xml version="1.1" encoding="UTF-8"?>
 <robot name="vektor" xmlns:xacro="http://www.ros.org/wiki/xacro">
-    <xacro:include filename="vektor_core.xacro"/>
-    <xacro:include filename="gazebo_control.xacro"/>
-    <xacro:include filename="lidar.xacro"/>
+    <xacro:include filename="components.xacro"/>
+    <xacro:include filename="plugins.xacro"/>
+    <!-- <xacro:include filename="lidar.xacro"/> -->
     <!-- <xacro:include filename="camera.xacro"/> -->
-    <xacro:include filename="depth_camera.xacro"/>
+    <!-- <xacro:include filename="depth_camera.xacro"/> -->
 </robot>
