Commit message: added base_footprint link

File: vektor_pkg/description/components.xacro (robot description, xacro)
@@ -1,8 +1,12 @@
 <?xml version="1.1" encoding="UTF-8"?>
 <robot xmlns:xacro="http://www.ros.org/wiki/xacro">
-  <!-- imports -->
   <xacro:include filename="inertial_macros.xacro"/>
   <xacro:include filename="materials.xacro"/>
-  <!-- links ans joints -->
+  <link name="base_footprint"/>
+  <joint name="base_joint" type="fixed">
+    <parent link="base_footprint"/>
+    <child link="base_link"/>
+    <origin xyz="0 0 0.05"/>
+  </joint>
   <link name="base_link"/>
   <joint name="chassis_joint" type="fixed">
@@ -32,5 +36,5 @@
     <parent link="base_link"/>
     <child link="left_wheel_link"/>
-    <origin xyz="0 0.175 0" rpy="-${pi/2} 0 0"/>
+    <origin xyz="0 0.17 0" rpy="-${pi/2} 0 0"/>
     <axis xyz="0 0 1"/>
   </joint>
@@ -54,5 +58,5 @@
     <parent link="base_link"/>
     <child link="right_wheel_link"/>
-    <origin xyz="0 -0.175 0" rpy="${pi/2} 0 0"/>
+    <origin xyz="0 -0.17 0" rpy="${pi/2} 0 0"/>
     <axis xyz="0 0 -1"/>
   </joint>
@@ -74,7 +78,7 @@
   </link>
   <joint name="caster_wheel_joint" type="fixed">
-    <parent link="chassis_link"/>
+    <parent link="base_link"/>
     <child link="caster_wheel_link"/>
-    <origin xyz="0.24 0 0"/>
+    <origin xyz="0.14 0 0"/>
   </joint>
   <link name="caster_wheel_link">
