Commit message: Added LiDAR sensor to simulation

File: vektor_pkg/description/lidar.xacro (robot description, xacro)
@@ -22,3 +22,33 @@
         </xacro:inertial_cylinder>
     </link>
+    <gazebo reference="lidar_frame">
+        <material>Gazebo/Green</material>
+        <sensor name="lidar" type="ray">
+            <pose> 0 0 0 0 0 0 </pose>
+            <visualize>true</visualize>
+            <update_rate>10</update_rate>
+            <ray>
+                <scan>
+                    <horizontal>
+                        <samples>360</samples>
+                        <resolution>1</resolution>
+                        <min_angle>-3.14</min_angle>
+                        <max_angle>3.14</max_angle>
+                    </horizontal>
+                </scan>
+                <range>
+                    <min>0.3</min>
+                    <max>12</max>
+                    <resolution>0.01</resolution>
+                </range>
+            </ray>
+            <plugin name="lidar_controller" filename="libgazebo_ros_ray_sensor.so">
+                <ros>
+                    <argument>~/out:=scan</argument>
+                </ros>
+                <output_type>sensor_msgs/LaserScan</output_type>
+                <frame_name>lidar_frame</frame_name>
+            </plugin>
+        </sensor>
+    </gazebo>
 </robot>

Commit message: lidar adjust

File: vektor_pkg/description/lidar.xacro (robot description, xacro)
@@ -2,5 +2,5 @@
 <robot xmlns:xacro="http://www.ros.org/wiki/xacro">
     <joint name="lidar_joint" type="fixed">
-        <parent link="chassis_link"/>
+        <parent link="base_link"/>
         <child link="lidar_frame"/>
         <origin xyz="0.1 0 0.175" rpy="0 0 0"/>
@@ -26,25 +26,31 @@
     </link>
     <gazebo reference="lidar_frame">
-        <sensor name='lidar_frame' type='gpu_lidar'>
+        <sensor name='my_lidar' type='gpu_lidar'>
             <pose>0 0 0 0 0 0</pose>
             <topic>lidar</topic>
             <ignition_frame_id>lidar_frame</ignition_frame_id>
             <update_rate>10</update_rate>
-            <ray>
+            <lidar>
                 <scan>
                     <horizontal>
-                        <samples>360</samples>
+                        <samples>640</samples>
                         <resolution>1</resolution>
                         <min_angle>-3.14</min_angle>
                         <max_angle>3.14</max_angle>
                     </horizontal>
+                    <vertical>
+                      <samples>1</samples>
+                      <resolution>1</resolution>
+                      <min_angle>0.0</min_angle>
+                      <max_angle>0.0</max_angle>
+                    </vertical>
                 </scan>
                 <range>
-                    <min>0.3</min>
-                    <max>5.0</max>
+                    <min>0.08</min>
+                    <max>10.0</max>
                     <resolution>0.01</resolution>
                 </range>
-            </ray>
-            <always_on>1</always_on>
+            </lidar>
+            <always_on>true</always_on>
             <visualize>true</visualize>
         </sensor>
