Commit message: project refactoring

File: vektor_description/urdf/sensors/lidar_sensor.xacro (robot description, xacro)
@@ -2,5 +2,5 @@
 <robot xmlns:xacro="http://www.ros.org/wiki/xacro">
   <xacro:macro name="lidar" params="prefix parent *origin">
-    <link name="${prefix}_link">
+    <link name="${prefix}_lidar_link">
       <visual>
         <geometry>
@@ -18,14 +18,14 @@
       </xacro:inertial_cylinder>
     </link>
-    <joint name="lidar_joint" type="fixed">
+    <joint name="${prefix}_lidar_joint" type="fixed">
       <parent link="${parent}" />
-      <child link="${prefix}_link" />
+      <child link="${prefix}_lidar_link" />
       <xacro:insert_block name="origin" />
     </joint>
-    <gazebo reference="${prefix}_link">
+    <gazebo reference="${prefix}_lidar_link">
       <sensor name='${prefix}_lidar' type='gpu_lidar'>
         <pose>0 0 0 0 0 0</pose>
-        <topic>scan</topic>
-        <ignition_frame_id>${prefix}_link</ignition_frame_id>
+        <topic>lidar</topic>
+        <ignition_frame_id>${prefix}_lidar_link</ignition_frame_id>
         <update_rate>10</update_rate>
         <lidar>

File: vektor_description/urdf/sensors/rgbd_camera_sensor.xacro (robot description, xacro)
@@ -26,5 +26,5 @@
       <sensor name="${prefix}_rgbd_camera" type="rgbd_camera">
         <update_rate>30</update_rate>
-        <topic>rgbd</topic>
+        <topic>camera</topic>
         <ignition_frame_id>${prefix}_rgbd_camera_link</ignition_frame_id>
         <camera>

File: vektor_description/urdf/structures/assembly.xacro (robot description, xacro)
@@ -1,7 +1,9 @@
 <?xml version="1.1" encoding="UTF-8"?>
 <robot xmlns:xacro="http://www.ros.org/wiki/xacro">
+  <xacro:include filename="materials.xacro" />
   <xacro:include filename="inertial_macro.xacro" />
-  <xacro:include filename="materials.xacro" />
-  <xacro:include filename="wheel_component.xacro" />
+  <xacro:include filename="wheel.xacro" />
+  <xacro:include filename="../sensors/lidar_sensor.xacro" />
+  <xacro:include filename="../sensors/rgbd_camera_sensor.xacro" />
   <link name="base_footprint" />
   <link name="base_link" />
@@ -34,11 +36,19 @@
     <origin xyz="-0.1 0 0" />
   </joint>
-  <xacro:wheel prefix="left" parent="base_link">
+  <xacro:wheel
+    prefix="left"
+    radius="0.05"
+    length="0.04"
+    parent="base_link">
     <origin xyz="0 0.17 0" rpy="-${pi/2} 0 0" />
-    <axis xyz="0 0 1"/>
+    <axis xyz="0 0 1" />
   </xacro:wheel>
-  <xacro:wheel prefix="right" parent="base_link">
+  <xacro:wheel
+      prefix="right"
+      radius="0.05"
+      length="0.04"
+      parent="base_link">
     <origin xyz="0 -0.17 0" rpy="${pi/2} 0 0" />
-    <axis xyz="0 0 -1"/>
+    <axis xyz="0 0 -1" />
   </xacro:wheel>
   <link name="caster_wheel_link">
@@ -63,4 +73,10 @@
     <origin xyz="0.14 0 0" />
   </joint>
+  <xacro:lidar prefix="main" parent="chassis_link">
+    <origin xyz="0.1 0 0.175" rpy="0 0 0" />
+  </xacro:lidar>
+  <xacro:rgbd_camera prefix="main" parent="base_link">
+    <origin xyz="0.205 0 0.075" rpy="0 0 0" />
+  </xacro:rgbd_camera>
   <gazebo reference="caster_wheel_link">
     <mu1 value="0.001" />

File: vektor_description/urdf/structures/wheel.xacro (robot description, xacro)
@@ -1,9 +1,9 @@
 <?xml version="1.1" encoding="UTF-8"?>
 <robot xmlns:xacro="http://www.ros.org/wiki/xacro">
-  <xacro:macro name="wheel" params="prefix parent *origin *axis">
+  <xacro:macro name="wheel" params="prefix radius length parent *origin *axis">
     <link name="${prefix}_wheel_link">
       <visual>
         <geometry>
-          <cylinder radius="0.05" length="0.04" />
+          <cylinder radius="${radius}" length="${length}" />
         </geometry>
         <material name="blue" />
@@ -11,8 +11,8 @@
       <collision>
         <geometry>
-          <cylinder radius="0.05" length="0.04" />
+          <cylinder radius="${radius}" length="${length}" />
         </geometry>
       </collision>
-      <xacro:inertial_cylinder mass="0.1" length="0.04" radius="0.05">
+      <xacro:inertial_cylinder mass="0.1" radius="${radius}" length="${length}">
         <origin xyz="0 0 0" rpy="0 0 0" />
       </xacro:inertial_cylinder>

File: vektor_description/urdf/vektor.xacro (robot description, xacro)
@@ -2,21 +2,20 @@
 <robot name="vektor" xmlns:xacro="http://www.ros.org/wiki/xacro">
   <xacro:arg name="ros2_control" default="false" />
-  <xacro:include filename="structures/base_component.xacro" />
-  <xacro:include filename="plugins/joint_state_publisher_plugin.xacro" />
-  <xacro:include filename="plugins/sensors_plugin.xacro" />
-  <xacro:include filename="sensors/lidar_sensor.xacro" />
-  <xacro:include filename="sensors/rgbd_camera_sensor.xacro" />
-  <xacro:lidar prefix="main" parent="chassis_link">
-    <origin xyz="0.1 0 0.175" rpy="0 0 0" />
-  </xacro:lidar>
-  <xacro:rgbd_camera prefix="main" parent="base_link">
-    <origin xyz="0.205 0 0.075" rpy="0 0 0" />
-  </xacro:rgbd_camera>
+  <xacro:arg name="vektor_simulation" default="$(find vektor_simulation)" />
+  <xacro:arg name="vektor_controllers" default="$(find vektor_controllers)" />
+  <xacro:include filename="structures/assembly.xacro" />
+  <xacro:include
+    filename="$(arg vektor_simulation)/plugins/joint_state_publisher_plugin.xacro" />
+  <xacro:include
+    filename="$(arg vektor_simulation)/plugins/sensors_plugin.xacro" />
   <xacro:if value="$(arg ros2_control)">
-    <xacro:include filename="plugins/ros2_control_plugin.xacro" />
-    <xacro:include filename="ros2_control/diff_drive_ros2_control.xacro" />
+    <xacro:include
+      filename="$(arg vektor_simulation)/plugins/ros2_control_plugin.xacro" />
+    <xacro:include
+      filename="$(arg vektor_controllers)/urdf/diff_drive_ros2_control.xacro" />
   </xacro:if>
   <xacro:unless value="$(arg ros2_control)">
-    <xacro:include filename="plugins/diff_drive_plugin.xacro" />
+    <xacro:include
+      filename="$(arg vektor_simulation)/plugins/diff_drive_plugin.xacro" />
   </xacro:unless>
 </robot>

File: vektor_simulation/plugins/ros2_control_plugin.xacro (robot description, xacro)
@@ -5,5 +5,5 @@
       filename="ign_ros2_control-system"
       name="ign_ros2_control::IgnitionROS2ControlPlugin">
-      <parameters>$(find vektor_description)/controllers/diff_drive_controller_velocity.yaml</parameters>
+      <parameters>$(find vektor_controllers)/config/vektor_controllers.yaml</parameters>
     </plugin>
   </gazebo>
